File: 2024KASAboard/2024KASAboard.kicad_sch (KiCad schematic)
At the start: 2 parts, among them U1 Pico, U2 BME280

Commit message: tamura
Connections:
- net at U2.3 (CSB): now also U1.25 (GPIO19)
Changed lines of the file:
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@@
+	(wire
+		(pts
+			(xy 209.55 97.79) (xy 153.67 97.79)
+		)
+		(stroke
+			(width 0)
+			(type default)
+		)
+	)
+	(wire
+		(pts
+			(xy 209.55 78.74) (xy 209.55 97.79)
+		)
+		(stroke
+			(width 0)
+			(type default)
+		)
+	)
 	(wire
 		(pts
